File: kicad-project-v1/wifi-guitar-extension.kicad_pcb (KiCad board)
At the start: 2 copper layers, 54.6 x 41.9 mm, 21 parts, among them IC1 ATMEGA88PA-A, P1 CONN_13X2, P2 CONN_4X2, P3 CONN_2, P4 CONN_10X2, U1 CS5343, X1 12.288MHz

Commit message: Added resistor pulling up the SDOUT line in CS534x (to ensure the Master Mode). Added optional connector for connecting the UART.
Parts:
- added K1: CONN_3, PIN_ARRAY_3X1, B.Cu at (30.5, 16.5)
- added R4: 10k, SM0805, F.Cu at (38.7, 39.4)
- P2: footprint pin_array_4x2 -> pin_array_4x2_reversed; moved to F.Cu
- renumbered R4 to R5, R5 to R6, R6 to R7, R7 to R8
Connections:
- P1 pad 10: (no net) -> /RPI_RXD
- P1 pad 8: (no net) -> /RPI_TXD
Routing:
- net /RPI_PCM_DIN: track 13.5 -> 16.7 mm
- net /RPI_TXD: track 0.00 -> 2.54 mm
- net /RPI_RXD: track 0.00 -> 2.54 mm
- net GND: track 166.2 -> 168.8 mm
- net /V3,3: track 147.8 -> 149.4 mm
Other:
- board size 54.6 x 41.9 mm -> 54.6 x 44.4 mm
- board text added: "Not needed if K1 is not mounted"
