File: kicad-project-v1/wifi-guitar-extension.sch (KiCad schematic (older format))
At the start: 21 parts, among them IC1 ATMEGA88PA-A, P1 CONN_13X2, P2 CONN_4X2, P3 CONN_2, P4 CONN_10X2, U1 CS5343, X1 12.288MHz

Commit message: Added resistor pulling up the SDOUT line in CS534x (to ensure the Master Mode). Added optional connector for connecting the UART.
Parts:
- added K1: CONN_3, ~, symbol CONN_3
- added R4: 10k, ~, symbol R
- renumbered R4 to R5, R5 to R6, R6 to R7, R7 to R8
Connections:
- net labels added: RPI_RXD, RPI_TXD
- wire segments 120 -> 127
Other:
- note added: "Please note, that P2 is mounted on the same side of PCB\nas P1, but pin numbers are located as it was mounted\non the oposite side!"
- note added: "Resistors configuring the ADC speed. For 48kHz sampling with\n12.288MHz crystal, we should select SSM with 256x multiplication\nfactor, so neither R5 nor R6 should be mounted.\nR4 should be mounted, as it enforces the Master Mode\n"
- note removed: "Please note, that P2 is mounted on the sime side of PCB\nas P1, but pin numbers are located as it was mounted\non the oposite side!"
- note removed: "Resistors configuring the ADC speed. For 48kHz sampling with\n12.288MHz crystal, we should select SSM with 256x multiplication\nfactor, so none of those resistors should be mounted\n"
- moved on the sheet: R5, R6
